File: kicad/host_shell.kicad_sch (KiCad schematic)
At the start: 151 parts, among them J1 Conn_02x12_Odd_Even, J2 Conn_01x02, J3 Conn_01x03, J4 Conn_01x02, J5 Micro_SD_Card_Det_Hirose_DM3AT, J6 Conn_01x02, J7 Conn_01x40, P1 TYPE-C16PIN, Q1 NPN, Q2 IRLML2246TRPBF, Q3 IRLML2246TRPBF, Q4 NMOS, SW1 TBD, SW12 TBD, SW13 TBD, SW14 TBD, SW15 TBD, SW16 TBD, SW17 TBD, SW18 TBD, SW2 TBD, SW3 TBD, SW4 TBD, SW5 TBD, SW6 TBD, SW7 TBD, U1 RP2350B, U10 MCP73831-2-OT, U11 TPS63802, U2 74AHC541, U3 W25Q32JVSSIQ, U5 PCA9555PW, U6 RT9080-33GJ5, U7 LM4890, U8 LM4890, U9 XC6194, Y1 ABM8-272-T3

Commit message: wip: schematics
Parts:
- removed C31, C32, C37: 1u, Capacitor_SMD:C_0603_1608Metric, symbol Device:C_Small
- removed C34, C38: 10u, Capacitor_SMD:C_0603_1608Metric, symbol Device:C_Small
- removed C35, C39: 100n, Capacitor_SMD:C_0402_1005Metric, symbol Device:C_Small
- removed JP1, JP2, JP3: SolderJumper_3_Bridged12, symbol Jumper:SolderJumper_3_Bridged12
- removed L4: TBD, symbol Device:L_Small
- removed Q1: NPN, symbol Simulation_SPICE:NPN
- removed Q2, Q3: IRLML2246TRPBF, symbol Simulation_SPICE:PMOS
- removed R35, R36, R37: 0, Resistor_SMD:R_0402_1005Metric, symbol Device:R_Small
- removed R43, R45: 22k, Resistor_SMD:R_0402_1005Metric, symbol Device:R_Small
- removed R49: 10k, Resistor_SMD:R_0402_1005Metric, symbol Device:R_Small
- added C22: 100n, Capacitor_SMD:C_0402_1005Metric, symbol Device:C_Small
- added C23, C24: 100u, symbol Device:C_Polarized_Small
- added C50: 100n, symbol Device:C_Small
- added C51, C52: 10n, Capacitor_SMD:C_0603_1608Metric, symbol Device:C_Small
- added C53, C54, C55, C56, C60, C61: 1u, Capacitor_SMD:C_0603_1608Metric, symbol Device:C_Small
- added C57, C58, C59: 100n, Capacitor_SMD:C_0603_1608Metric, symbol Device:C_Small
- added J8: AudioJack3_SwitchTR, symbol Connector_Audio:AudioJack3_SwitchTR
- added JP1, JP2, JP3: SolderJumper_3_Bridged12, symbol shpc_mechanical:SolderJumper_3_Bridged12
- added Q1, Q3, Q7: BSS138, Package_TO_SOT_SMD:SOT-23, symbol Transistor_FET:BSS138
- added Q2: BSS84, Package_TO_SOT_SMD:SOT-23, symbol Transistor_FET:BSS84
- added Q5, Q6: IRLML2246TRPBF, symbol Transistor_FET:Q_PMOS_GSD
- added R34: 1k, symbol Device:R_Small
- added R56: 1k, Resistor_SMD:R_0402_1005Metric, symbol Device:R_Small
- added R59, R60: 2.2k, Resistor_SMD:R_0402_1005Metric, symbol Device:R_Small
- added R61, R62, R68, R69, R70, R71: 22k, Resistor_SMD:R_0402_1005Metric, symbol Device:R_Small
- added R63, R64, R65: 100k, Resistor_SMD:R_0402_1005Metric, symbol Device:R_Small
- added R66, R67: 10k, Resistor_SMD:R_0402_1005Metric, symbol Device:R_Small
- added TP14, TP15, TP16, TP17, TP18: TestPoint_Small, TestPoint:TestPoint_Pad_D1.0mm, symbol Connector:TestPoint_Small
- added U12: SN74LVC1G18, Package_TO_SOT_SMD:SOT-23-6, symbol shpc_ic:SN74LVC1G18
- added U13: LM4880, symbol shpc_ic:LM4880
- added U4: SN74LVC1G18, Package_TO_SOT_SMD:SOT-23-6, symbol shpc_ic:74LVC2G17
- C41: value 4.7u -> 10u
- C49: value TBD -> 100n; footprint Capacitor_SMD:C_0603_1608Metric -> (none); LCSC C15849 -> (none); URL https://www.lcsc.com/product-detail/C15849.html -> (none)
- Q4: value NMOS -> BSS138W
- R30: value 0 -> 1M; footprint Resistor_SMD:R_0402_1005Metric -> (none); LCSC C17168 -> (none); URL https://www.lcsc.com/product-detail/C17168.html -> (none)
- R31: value 0 -> 100k; footprint Resistor_SMD:R_0402_1005Metric -> (none); LCSC C17168 -> (none); URL https://www.lcsc.com/product-detail/C17168.html -> (none); now fitted
- R32: value 0 -> 1k; footprint Resistor_SMD:R_0402_1005Metric -> (none); LCSC C17168 -> (none); URL https://www.lcsc.com/product-detail/C17168.html -> (none); now fitted
- R52, R53, R54: value 100 -> 22
Connections:
- net HSLCD_IM0 is gone; now on net 3V3: J7.38 (Pin_38)
- net HSLCD_IM1 is gone; now on net 3V3: J7.39 (Pin_39)
- net HSLCD_IM2 is gone; now on net HSLCD_SPIEN: J7.40 (Pin_40)
- net HSTF_MOSI is gone; now on net HSSPI_MOSI: J5.3 (CMD), U1.44 (GPIO35), U2.15 (Y3)
- net LC3V3 is gone; now on net 3V3: J1.23 (Pin_23)
- net 3V3: now also C49.1, J7.33 (Pin_33), R19.1, R20.1, JP1.1 (A), JP2.3 (B), JP3.3 (B), U12.5 (V_{CC}); no longer R19.2, R20.2
- net A3V3: now also R30.1, R31.1, C50.1, C57.2, C58.1, C59.1, U13.8 (VDD), U4.5 (V_{CC})
- net GND: now also C36.1, R32.2, C22.2, C50.2, C51.1, C52.2, C57.1, C58.2, C59.2, C60.2, C61.2, J8.S, JP1.3 (B), JP2.1 (A), JP3.1 (A), Q1.2 (S), Q3.2 (S), Q7.2 (S), R34.1, R63.2, R64.2, R67.2, U12.2 (GND), U13.4 (GND), U4.2 (GND); no longer R31.2
- net HSAUX_SCL: now also R15.2; no longer R20.1
- net HSAUX_SDA: now also R16.2; no longer R19.1
- net HSLCD_BL: now also R56.1; no longer Q4.2 (G), R55.1
- net HSLCD_CS: now also U1.23 (GPIO23); no longer U1.28 (GPIO27)
- net HSLCD_D0: now also U1.11 (GPIO12); no longer U1.16 (GPIO16)
- net HSLCD_D1: now also U1.12 (GPIO13); no longer U1.17 (GPIO17)
- net HSLCD_D2: now also U1.13 (GPIO14); no longer U1.18 (GPIO18)
- net HSLCD_D3: now also U1.14 (GPIO15); no longer U1.19 (GPIO19)
- net HSLCD_D4: now also U1.16 (GPIO16); no longer U1.20 (GPIO20)
- net HSLCD_D5: now also U1.17 (GPIO17); no longer U1.21 (GPIO21)
- net HSLCD_D6: now also U1.18 (GPIO18); no longer U1.22 (GPIO22)
- net HSLCD_D7: now also U1.19 (GPIO19); no longer U1.23 (GPIO23)
- net HSLCD_DC: now also U1.20 (GPIO20), U12.6 (Y0); no longer J7.10 (Pin_10), U1.25 (GPIO24)
- net HSLCD_RD: now also U1.22 (GPIO22); no longer U1.27 (GPIO26)
- net HSLCD_RST: now also U1.25 (GPIO24); no longer U1.14 (GPIO15)
- net HSLCD_WR: now also U1.21 (GPIO21); no longer U1.26 (GPIO25)
- net LCAUDIO_L: now also R70.1; no longer RV1.3A
- net LCAUDIO_R: now also R71.1; no longer RV1.3B
- net LCAUX_SCL: now also R19.2; no longer R16.2
- net LCAUX_SDA: now also R20.2; no longer R15.2
- net LCVSYS: now also Q6.3 (D)
- net MUTEX: now also U5.19 (IO1_6); no longer U7.1 (~{SD}), U8.1 (~{SD})
- net VBAT: now also Q2.3 (D), Q5.3 (D), R65.1
- net VBUS: now also Q5.1 (G)
- net VCOM: now also Q5.2 (S)
- net VSYS: now also Q3.1 (G), Q6.2 (S), R64.1
- net at R51.2: now also Q1.3 (D), Q6.1 (G)
- net at J7.1 (Pin_1): now also TP14.1
- net HSSPI_MOSI: now reaches J7.13 (Pin_13)
- net at J7.14 (Pin_14): now also TP18.1
- net at J7.2 (Pin_2): now also TP15.1
- net at J7.3 (Pin_3): now also TP16.1
- net at J7.4 (Pin_4): now also TP17.1
- net at RV1.2A: now also C53.2, C55.2
- net at RV1.2B: now also C54.2, C56.2; no longer C36.1
- net at U5.3 (A2): now also JP3.2 (C)
- net at R13.1: now also U1.26 (GPIO25); no longer U1.11 (GPIO12)
- net at R14.1: now also U1.27 (GPIO26); no longer U1.12 (GPIO13)
- net ADCBAT: now reaches U1.49 (GPIO40/ADC0)
- net ADCBAT: now also C22.1, R66.2, R67.1
- net HSAUDIO_L: now reaches U1.57 (GPIO46/ADC6)
- net HSAUDIO_L: now also U4.1 (1A)
- net HSAUDIO_R: now reaches U1.58 (GPIO47/ADC7)
- net HSAUDIO_R: now also U4.3 (2A)
- net at C33.2, R44.1, U7.4 (-IN): now also C53.1
- net at U7.2 (BYPASS), U7.3 (+IN): now also C60.1
- net at C36.2: now also U13.3 (BYP)
- net at C40.2, R46.1, U8.4 (-IN): now also C54.1
- net at U8.2 (BYPASS), U8.3 (+IN): now also C61.1
- net LCVSYSEN: now reaches U5.18 (IO1_5)
- net LCVSYSEN: now also Q1.1 (G), R63.1
- net at U5.2 (A1): now also JP2.2 (C); no longer R32.2
- net HSLCD_SPIEN: now reaches U5.20 (IO1_7)
- net HSLCD_SPIEN: now also U12.1 (S)
- net +3V3: no longer names the net of R32.1
- net +3V3: now also C24.2, J8.R; no longer R30.1
- net HSTF_MISO renamed HSSPI_MISO
- net HSTF_SCK renamed HSSPI_SCK
- net HSSPI_SCK: now also U12.4 (Y1)
- new net: C52.1, R59.2, R61.1
- new net: Q4.2 (G), R55.1, R56.2
- new net: C56.1, R68.1, U13.6 (INB)
- new net: C23.2, J8.T, R34.2
- new net: JP1.2 (C), U5.21 (A0)
- new net: C24.1, R68.2, U13.7 (OUTB)
- new net: R61.2, R70.2, RV1.3A
- new net: C23.1, R69.2, U13.1 (OUTA)
- new net: C55.1, R69.1, U13.2 (INA)
- new net: Q7.3 (D), R31.2, U13.5 (~{SD})
- new net: R60.1, U4.4 (2Y)
- new net: R59.1, U4.6 (1Y)
- new net: C51.2, R60.2, R62.1
- new net: Q2.1 (G), Q3.3 (D), R65.2
- new net: Q2.2 (S), R66.1
- new net: R62.2, R71.2, RV1.3B
- new net HSLCD_DCCK: J7.10 (Pin_10), U12.3 (A)
- new net SPKEN: J8.RN, Q7.1 (G), R30.2, U7.1 (~{SD}), U8.1 (~{SD})
- no-connect marks 32 -> 23
Other:
- moved on the sheet: C33, C40, J2, J4, L3, Q4, R44, R46, R52, R53, R54, R55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

Commit message: wip
Parts:
- removed C29, C30: 1u, Capacitor_SMD:C_0402_1005Metric, symbol Device:C_Small
- removed C41: 10u, Capacitor_SMD:C_0603_1608Metric, symbol Device:C_Small
- removed C42: 10u, symbol Device:C_Small
- removed J5: Micro_SD_Card_Det_Hirose_DM3AT, Connector_Card:microSD_HC_Hirose_DM3AT-SF-PEJM5, symbol Connector:Micro_SD_Card_Det_Hirose_DM3AT
- removed R25: 1k, Resistor_SMD:R_0402_1005Metric, symbol Device:R_Small
- removed SW1, SW16, SW17: TBD, Button_Switch_SMD:SW_Push_1P1T_NO_Vertical_Wuerth_434133025816, symbol shpc_mechanical:SKRPACE010
- removed TP9: TestPoint_Small, TestPoint:TestPoint_Pad_D1.0mm, symbol Connector:TestPoint_Small
- removed U6: RT9080-33GJ5, Package_TO_SOT_SMD:TSOT-23-5, symbol shpc_ic:RT9080-33GJ5
- added C25: 4.7u, Capacitor_SMD:C_0603_1608Metric, symbol Device:C_Small
- added C26, C62, C63: 100n, Capacitor_SMD:C_0402_1005Metric, symbol Device:C_Small
- added C64: 22u, Capacitor_SMD:C_0603_1608Metric, symbol Device:C_Small
- added C65: 10n, Capacitor_SMD:C_0603_1608Metric, symbol Device:C_Small
- added C66, C67, C68, C69: 10u, Capacitor_SMD:C_0603_1608Metric, symbol Device:C_Small
- added D7, D8: TBD, symbol Device:LED_Small
- added J10: Conn_02x10_Odd_Even, symbol Connector_Generic:Conn_02x10_Odd_Even
- added J11, J5: Conn_01x02, shpc_mechanical:SolderWirePad_1x02_SMD_150x50mil, symbol Connector_Generic:Conn_01x02
- added J9: Micro_SD_Card_Det2, Connector_Card:microSD_HC_Hirose_DM3AT-SF-PEJM5, symbol shpc_mechanical:Micro_SD_Card_Det2
- added JP4: SolderJumper_3_Bridged12, Jumper:SolderJumper-3_P1.3mm_Bridged12_RoundedPad1.0x1.5mm, symbol shpc_mechanical:SolderJumper_3_Bridged12
- added R35, R73: 33, Resistor_SMD:R_0402_1005Metric, symbol Device:R_Small
- added R36: 1k, Resistor_SMD:R_0402_1005Metric, symbol Device:R_Small
- added R43, R45, R72, R74: 10k, Resistor_SMD:R_0402_1005Metric, symbol Device:R_Small
- added TP19, TP20, TP21, TP22, TP23, TP24, TP25, TP26, TP27, TP28, TP29, TP30, TP31, TP32, TP33, TP34, TP35, TP36, TP37, TP38, TP39, TP40, TP41, TP42, TP43, TP44, TP45, TP46, TP47, TP48, TP49, TP50, TP51: TestPoint_Small, TestPoint:TestPoint_Pad_D1.0mm, symbol Connector:TestPoint_Small
- added U14: APS6404L-3SQRx-SN, Package_SO:SOP-8_3.76x4.96mm_P1.27mm, symbol Memory_RAM:APS6404L-3SQRx-SN
- C1, C49, C50: LCSC (none) -> C1525
- C22: LCSC C1548 -> C1525
- C23, C24: value 100u -> 220u; footprint (none) -> Capacitor_SMD:CP_Elec_6.3x5.4; LCSC (none) -> C3345
- C43: footprint (none) -> Capacitor_SMD:C_0603_1608Metric; LCSC (none) -> C1691
- C45: footprint Capacitor_SMD:C_0402_1005Metric -> Capacitor_SMD:C_0603_1608Metric; LCSC C52923 -> C1691
- C46: footprint Capacitor_SMD:C_0402_1005Metric -> Capacitor_SMD:C_0603_1608Metric; LCSC C52923 -> C59461
- C47, C48: LCSC C52923 -> C1525
- C53, C54, C55, C56, C60, C61: LCSC C1691 -> C15849
- D4: value 1N4148WS -> SM4007PL; footprint (none) -> Diode_SMD:D_SOD-123F; LCSC (none) -> C64898
- D6: value LED_Small -> TBD
- J2, J4: now left out of the parts list
- J6: value Conn_01x02 -> FG PH-2AWT; footprint (none) -> Connector_JST:JST_PH_S2B-PH-SM4-TB_1x02-1MP_P2.00mm_Horizontal; LCSC (none) -> C2763693
- JP1, JP2, JP3: footprint (none) -> Jumper:SolderJumper-3_P1.3mm_Bridged12_RoundedPad1.0x1.5mm
- L3: footprint (none) -> Inductor_SMD:L_Sunlord_SWPA4018S
- Q1, Q3, Q7: value BSS138 -> BSS138W; footprint Package_TO_SOT_SMD:SOT-23 -> Package_TO_SOT_SMD:SOT-323_SC-70; LCSC (none) -> C504052
- Q2: value BSS84 -> BSS84W; footprint Package_TO_SOT_SMD:SOT-23 -> Package_TO_SOT_SMD:SOT-323_SC-70; LCSC (none) -> C919394
- Q4: footprint (none) -> Package_TO_SOT_SMD:SOT-323_SC-70; LCSC (none) -> C504052
- Q5, Q6: footprint (none) -> Package_TO_SOT_SMD:SOT-23; LCSC (none) -> C127272
- R1, R10, R11, R12, R13, R14, R2, R3, R4, R5, R6, R7, R8, R9: footprint (none) -> Resistor_SMD:R_0402_1005Metric; LCSC (none) -> C25118
- R15, R16, R19, R20: footprint (none) -> Resistor_SMD:R_0402_1005Metric; LCSC (none) -> C25900
- R17, R18: footprint (none) -> Resistor_SMD:R_0402_1005Metric; LCSC (none) -> C25092
- R21, R38: footprint (none) -> Resistor_SMD:R_0402_1005Metric; LCSC (none) -> C25744
- R24, R33: URL (none) -> -- ミックスされた値 --
- R30: footprint (none) -> Resistor_SMD:R_0402_1005Metric; LCSC (none) -> C26083
- R31: footprint (none) -> Resistor_SMD:R_0402_1005Metric; LCSC (none) -> C25741
- R32, R34: footprint (none) -> Resistor_SMD:R_0402_1005Metric; LCSC (none) -> C11702
- R39: LCSC C17168 -> C25885
- R40, R66, R67: LCSC C17168 -> C25744; URL https://www.lcsc.com/product-detail/C17168.html -> -- ミックスされた値 --
- R41: LCSC C17168 -> C1161
- R42: LCSC C17168 -> C64042
- R48, R50: LCSC C25768 -> C25744; URL https://www.lcsc.com/product-detail/C25768.html -> -- ミックスされた値 --
- R51, R55, R63, R64, R65: LCSC C17168 -> C25741
- R52, R53, R54: LCSC C25768 -> C25092
- R56: LCSC C25768 -> C11702; URL https://www.lcsc.com/product-detail/C25768.html -> -- ミックスされた値 --
- R59, R60: LCSC C25768 -> C25879
- R61, R62, R70, R71: value 22k -> 10k; LCSC C25768 -> C25744; URL https://www.lcsc.com/product-detail/C25768.html -> -- ミックスされた値 --
- SW12, SW13, SW14, SW15, SW18, SW3, SW4, SW5, SW6: value TBD -> Rubber; footprint Button_Switch_SMD:SW_Push_1P1T_NO_Vertical_Wuerth_434133025816 -> shpc_mechanical:Rubber_Contact; LCSC C139797 -> (none); now not fitted; now left out of the parts list
- SW2: value TBD -> SKRPACE010_6
- SW7: value TBD -> GT-TC018A-H0375-L1; footprint Button_Switch_SMD:SW_Push_1P1T_NO_Vertical_Wuerth_434133025816 -> shpc_mechanical:GT-TC018A-H0375-L1; LCSC C139797 -> C963235
- U1: LCSC (none) -> C42415655
- U10: LCSC (none) -> C14879
- U12: value SN74LVC1G18 -> SN74LVC1G18DBVR-TP; LCSC (none) -> C49333182
- U13: value LM4880 -> LM4880MX/NOPB; footprint (none) -> Package_SO:SOIC-8_3.9x4.9mm_P1.27mm
- U2: value 74AHC541 -> SN74AHC541PWR; footprint (none) -> Package_SO:TSSOP-20-1EP_4.4x6.5mm_P0.65mm_EP2.15x3.35mm; LCSC (none) -> C406865
- U4: value SN74LVC1G18 -> 74LVC2G17GW; footprint Package_TO_SOT_SMD:SOT-23-6 -> Package_TO_SOT_SMD:SOT-363_SC-70-6; LCSC (none) -> C19829576
- U7, U8: value LM4890 -> LM4890S
- U9: value XC6194 -> XC6194AA03ER-G; LCSC (none) -> C18221112
Connections:
- net LCGND is gone; now on net GND: J1.3 (Pin_3)
- net MUTEX is gone; now on net LCVSYSEN: U5.19 (IO1_6)
- net 3V3: now also C58.1, C59.1, FB2.1, R38.1, U7.6 (VDD), U8.6 (VDD), C25.1, C26.1, C67.1, C68.1, C69.1, J10.17 (Pin_17), J9.4 (VDD), R35.1, R43.1, R45.1, R74.1, U14.8 (VDD); no longer C15.1, R38.2, U1.59 (ADC_AVDD)
- net 3V3PG: now also TP41.1
- net A3V3: now also FB2.2, C62.1, C64.1, R73.1; no longer C50.1, C58.1, C59.1, U4.5 (V_{CC}), U7.6 (VDD), U8.6 (VDD)
- net ADCBAT: now also U1.54 (GPIO43/ADC3); no longer U1.49 (GPIO40/ADC0)
- net GND: now also C50.1, C25.2, C26.2, C62.2, C63.2, C64.2, C65.1, C66.1, C67.2, C68.2, C69.2, D8.1 (K), J10.1 (Pin_1), J10.20 (Pin_20), J11.2 (Pin_2), J5.2 (Pin_2), J9.6 (VSS), J9.9 (DET_B), J9.SH (SHIELD), JP4.1 (A), R72.2, U14.4 (VSS); no longer C50.2, U11.2 (MODE)
- net HSAUDIO_L: now also U1.55 (GPIO44/ADC4), TP19.1; no longer U1.57 (GPIO46/ADC6)
- net HSAUDIO_R: now also U1.56 (GPIO45/ADC5), TP20.1; no longer U1.58 (GPIO47/ADC7)
- net HSAUX_SCL: now also R20.2, TP32.1; no longer R15.2
- net HSAUX_SDA: now also R19.2, TP31.1; no longer R16.2
- net HSLCD_BL: now also U1.57 (GPIO46/ADC6), TP21.1
- net HSLCD_D0: now also J10.3 (Pin_3)
- net HSLCD_D1: now also J10.4 (Pin_4)
- net HSLCD_D2: now also J10.5 (Pin_5)
- net HSLCD_D3: now also J10.6 (Pin_6)
- net HSLCD_D4: now also J10.7 (Pin_7)
- net HSLCD_D5: now also J10.8 (Pin_8)
- net HSLCD_D6: now also J10.9 (Pin_9)
- net HSLCD_D7: now also J10.10 (Pin_10)
- net HSLCD_DC: now also J10.11 (Pin_11)
- net HSLCD_SPIEN: now also TP50.1
- net HSLCD_VSYNC: now also U1.28 (GPIO27), TP30.1
- net HSSPI_MISO: now also J7.14 (Pin_14), TP18.1, J9.7 (DAT0), R45.2, TP27.1
- net HSSPI_MOSI: now also J9.3 (CMD), TP24.1
- net HSSPI_SCK: now also J9.5 (CLK), TP25.1
- net LCAUX_SCL: now also R16.2; no longer R19.2
- net LCAUX_SDA: now also R15.2; no longer R20.2
- net LCTF_ENX: now also U5.17 (IO1_4), TP45.1; no longer U1.47 (GPIO38)
- net LCUSB_DM: now also TP34.1
- net LCUSB_DP: now also TP33.1
- net LCVSYSEN: now also TP49.1; no longer U5.18 (IO1_5)
- net SPKEN: now also Q7.3 (D), R31.2, U13.5 (SD); no longer J8.RN, Q7.1 (G), R30.2
- net SYSPG: now also TP40.1
- net SYSSD: now also U1.48 (GPIO39), C63.1, R72.1, TP29.1
- net VSYS: now also J10.2 (Pin_2), JP4.3 (B), TP39.1; no longer FB2.1
- net at U1.52 (GPIO41/ADC1): now also TP42.1
- net at U1.53 (GPIO42/ADC2): now also TP43.1
- net QSPI_D3: now reaches U1.70 (QSPI_SD3), U3.7 (~{HOLD}/~{RESET}/IO_{3})
- net QSPI_D3: now also U14.7 (SIO3)
- net QSPI_SCLK: now reaches U1.71 (QSPI_SCLK), U3.6 (CLK)
- net QSPI_SCLK: now also U14.6 (SCLK)
- net QSPI_D0: now reaches U1.72 (QSPI_SD0), U3.5 (DI/IO_{0})
- net QSPI_D0: now also U14.5 (SI/SIO0)
- net QSPI_D2: now reaches U1.73 (QSPI_SD2), U3.3 (~{WP}/IO_{2})
- net QSPI_D2: now also U14.3 (SIO2)
- net QSPI_D1: now reaches U1.74 (QSPI_SD1), U3.2 (DO/IO_{1})
- net QSPI_D1: now also U14.2 (SO/SIO1)
- net FLASH_CSX: now reaches U1.75 (~{QSPI_SS}), U3.1 (~{CS})
- net FLASH_CSX: now also R36.2
- net at U5.14 (IO1_1): now also J5.1 (Pin_1)
- net at U5.13 (IO1_0): now also J11.1 (Pin_1)
- net at U5.16 (IO1_3): now also TP44.1
- net BTN_D: now reaches SW3.1, U5.7 (IO0_3)
- net BTN_D: now also R36.1
- net at J1.4 (Pin_4): now also TP48.1
- net HSLCD_CS renamed HSLCD_CSX
- net HSLCD_CSX: now also U1.25 (GPIO24), J10.15 (Pin_15), TP38.1; no longer U1.23 (GPIO23)
- net HSLCD_RD renamed HSLCD_RDX
- net HSLCD_RDX: now also J10.13 (Pin_13), TP36.1
- net HSLCD_RST renamed HSLCD_RSTX
- net HSLCD_RSTX: now also U1.21 (GPIO21), J10.12 (Pin_12), TP35.1; no longer U1.25 (GPIO24)
- net HSLCD_WR renamed HSLCD_WRX
- net HSLCD_WRX: now also U1.23 (GPIO23), J10.14 (Pin_14), TP37.1; no longer U1.21 (GPIO21)
- net HSTF_CS renamed HSTF_CSX
- net HSTF_CSX: now also R38.2, D7.1 (K), J9.2 (DAT3/CD), TP26.1; no longer R38.1
- net LCTF_CS renamed LCTF_CSX
- new net: J9.10 (DET_A), TP51.1
- new net: D8.2 (A), R74.2
- new net: J10.18 (Pin_18), TP47.1
- new net: J10.19 (Pin_19), TP46.1
- new net: C65.2, J8.RN, Q7.1 (G), R30.2
- new net: D7.2 (A), R43.2
- new net: TP28.1, U1.47 (GPIO38)
- new net: TP22.1, U1.49 (GPIO40/ADC0)
- new net: C50.2, C66.2, R73.2, U4.5 (V_{CC})
- new net: JP4.2 (C), U11.2 (MODE)
- new net ADC_AVDD: C15.1, R35.2, U1.59 (ADC_AVDD)
- new net EXTVIDENX: J10.16 (Pin_16), U5.18 (IO1_5)
- new net PSRAM_CSX: TP23.1, U1.58 (GPIO47/ADC7), U14.1 (~{CE})
- no-connect marks 23 -> 18
Other:
- note added: "Note: If switching noise affects the audio, set MODE to High (PWM mode)."
- moved on the sheet: C10, C11, C12, C13, C14, C15, C16, C19, C2, C20, C21, C22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

Commit message: wip
Parts:
- removed J10: Conn_02x10_Odd_Even, symbol Connector_Generic:Conn_02x10_Odd_Even
- removed TP48: TestPoint_Small, TestPoint:TestPoint_Pad_D1.0mm, symbol Connector:TestPoint_Small
- added J5: Conn_02x10_Odd_Even, Connector_PinSocket_2.54mm:PinSocket_2x10_P2.54mm_Horizontal, symbol Connector_Generic:Conn_02x10_Odd_Even
- C35: renamed from C50; footprint (none) -> Capacitor_SMD:C_0402_1005Metric
- C55: renamed from C49; footprint (none) -> Capacitor_SMD:C_0402_1005Metric
- C56: renamed from C1; footprint (none) -> Capacitor_SMD:C_0402_1005Metric
- D3: renamed from D6; value TBD -> YLED0402R; footprint (none) -> LED_SMD:LED_0402_1005Metric_Pad0.77x0.64mm_HandSolder; LCSC (none) -> C21260817
- D5: renamed from D8; value TBD -> YLED0402B; footprint (none) -> LED_SMD:LED_0402_1005Metric_Pad0.77x0.64mm_HandSolder; LCSC (none) -> C30584803
- D6: renamed from D7; value TBD -> YLED0402Y; footprint (none) -> LED_SMD:LED_0402_1005Metric_Pad0.77x0.64mm_HandSolder; LCSC (none) -> C20608782
- J11: renamed from J1; footprint (none) -> shpc_mechanical:PinSocket_2x12_P2.54mm_Horizontal; now left out of the parts list
- J4: renamed from J7; footprint (none) -> Connector_FFC-FPC:TE_4-1734839-0_1x40-1MP_P0.5mm_Horizontal; now left out of the parts list
- J8: footprint (none) -> shpc_mechanical:Jack_3.5mm_PJ-316A-6A_Horizontal; LCSC (none) -> C128987
- SW10: renamed from SW15; now fitted
- SW2: renamed from SW6; now fitted
- SW3: renamed from SW5; now fitted
- SW4: now fitted
- SW5: renamed from SW3; now fitted
- SW6: renamed from SW18; now fitted
- SW7: renamed from SW12; now fitted
- SW8: renamed from SW13; now fitted
- SW9: renamed from SW14; now fitted
- U10: renamed from U13; LCSC (none) -> C2872533
- U2: renamed from U9; footprint (none) -> shpc_ic:USP-8B06
- U3: renamed from U11; footprint (none) -> shpc_ic:TPS63802; LCSC (none) -> C2845237
- renumbered C43 to C1, C64 to C10, C28 to C11, C18 to C12, C17 to C13, C25 to C14, C26 to C15, C4 to C16, C5 to C17, C16 to C18, C2 to C19, C44 to C2, C15 to C20, C3 to C21, C14 to C22, C8 to C23, C9 to C24, C10 to C25, C11 to C26, C12 to C27, C13 to C28, C20 to C29, C63 to C3, C21 to C30, C6 to C31, C7 to C32, C19 to C33, C66 to C34, C52 to C36, C51 to C37, C60 to C38, C53 to C39, C22 to C4, C67 to C40, C59 to C41, C33 to C42, C55 to C43, C56 to C44, C36 to C45, C57 to C46, C23 to C47, C24 to C48, C65 to C49, C45 to C5, C61 to C50, C54 to C51, C68 to C52, C58 to C53, C40 to C54, C69 to C57, C47 to C6, C48 to C7, C46 to C8, C62 to C9, FB2 to FB1, J6 to J1, J9 to J10, J5 to J2, J11 to J3, J3 to J6, J2 to J7, J4 to J9, JP4 to JP1, JP1 to JP2, JP2 to JP3, JP3 to JP4, L3 to L1, L1 to L2, Q5 to Q1, Q1 to Q2, Q6 to Q3, Q3 to Q4, Q2 to Q5, Q7 to Q6, Q4 to Q7, R28 to R1, R64 to R10, R65 to R11, R66 to R12, R67 to R13, R50 to R14, R42 to R15, R41 to R16, R74 to R17, R52 to R18, R53 to R19, R29 to R2, R54 to R20, R36 to R21, R33 to R22, R26 to R23, R27 to R24, R24 to R25, R22 to R26, R23 to R27, R35 to R28, R17 to R29, R39 to R3, R18 to R30, R20 to R31, R19 to R32, R1 to R33, R2 to R34, R3 to R35, R4 to R36, R5 to R37, R6 to R38, R7 to R39, R47 to R4, R8 to R40, R9 to R41, R10 to R42, R11 to R43, R12 to R44, R13 to R45, R14 to R46, R16 to R47, R15 to R48, R73 to R49, R40 to R5, R59 to R50, R60 to R51, R70 to R52, R61 to R53, R62 to R54, R71 to R55, R44 to R56, R69 to R57, R68 to R58, R34 to R59, R48 to R6, R32 to R60, R30 to R61, R31 to R62, R46 to R63, R56 to R64, R55 to R65, R21 to R66, R43 to R67, R38 to R68, R45 to R69, R72 to R7, R63 to R8, R51 to R9, SW7 to SW1, SW2 to SW11, TP11 to TP1, TP14 to TP10, TP15 to TP11, TP16 to TP12, TP17 to TP13, TP18 to TP14, TP47 to TP15, TP46 to TP16, TP22 to TP17, TP19 to TP18, TP20 to TP19, TP12 to TP2, TP21 to TP20, TP23 to TP21, TP10 to TP22, TP42 to TP23, TP43 to TP24, TP13 to TP25, TP28 to TP26, TP29 to TP27, TP35 to TP28, TP36 to TP29, TP40 to TP3, TP37 to TP30, TP38 to TP31, TP30 to TP32, TP27 to TP33, TP26 to TP34, TP25 to TP35, TP24 to TP36, TP33 to TP37, TP34 to TP38, TP31 to TP39, TP39 to TP4, TP32 to TP40, TP51 to TP41, TP41 to TP5, TP44 to TP6, TP45 to TP7, TP49 to TP8, TP50 to TP9, U10 to U1, U8 to U11, U2 to U13, U5 to U4, U3 to U5, U14 to U6, U1 to U7, U4 to U8, U7 to U9
Connections:
- net 3V3: now also J5.17 (Pin_17)
- net EXTVIDENX: now also J5.16 (Pin_16)
- net GND: now also U2.EP, J5.1 (Pin_1), J5.20 (Pin_20)
- net HSLCD_CSX: now also J5.15 (Pin_15)
- net HSLCD_D0: now also J5.3 (Pin_3)
- net HSLCD_D1: now also J5.4 (Pin_4)
- net HSLCD_D2: now also J5.5 (Pin_5)
- net HSLCD_D3: now also J5.6 (Pin_6)
- net HSLCD_D4: now also J5.7 (Pin_7)
- net HSLCD_D5: now also J5.8 (Pin_8)
- net HSLCD_D6: now also J5.9 (Pin_9)
- net HSLCD_D7: now also J5.10 (Pin_10)
- net HSLCD_DC: now also J5.11 (Pin_11)
- net HSLCD_RDX: now also J5.13 (Pin_13)
- net HSLCD_RSTX: now also J5.12 (Pin_12)
- net HSLCD_WRX: now also J5.14 (Pin_14)
- net VSYS: now also J5.2 (Pin_2)
- net at TP15.1: now also J5.18 (Pin_18)
- net at TP16.1: now also J5.19 (Pin_19)
- net LCALG0: now reaches TP17.1, U7.49 (GPIO40/ADC0)
- net LCALG0: now also J11.4 (Pin_4)
Other:
- moved on the sheet: TP15, TP16, TP17

Commit message: wip
Connections:
- net LCALG0 renamed LCA0
Changed lines of the file:
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@@
 		)
 	)
-	(label "LCALG0"
+	(label "LCA0"
 		(at 360.68 210.82 0)
 		(effects
@@
 		)
 	)
-	(label "LCALG0"
+	(label "LCA0"
 		(at 93.98 223.52 0)
 		(effects

Commit message: schematic review feedback
Parts:
- removed TP41, TP6, TP7: TestPoint_Small, TestPoint:TestPoint_Pad_D1.0mm, symbol Connector:TestPoint_Small
- added C58: 10u, Capacitor_SMD:C_0603_1608Metric, symbol Device:C_Small
- added C59: 100n, Capacitor_SMD:C_0402_1005Metric, symbol Device:C_Small
- added D7: LBAT54HT1G, Diode_SMD:D_SOD-323, symbol Device:D_Schottky_Small
- added R70, R74: 10k, Resistor_SMD:R_0402_1005Metric, symbol Device:R_Small
- added R71, R72: 100k, Resistor_SMD:R_0402_1005Metric, symbol Device:R_Small
- added R73: 47, Resistor_SMD:R_0402_1005Metric, symbol Device:R_Small
- added SW12, SW13: Rubber, shpc_mechanical:Rubber_Contact, symbol shpc_mechanical:SKRPACE010
- D4: value SM4007PL -> SS14; footprint Diode_SMD:D_SOD-123F -> Diode_SMD:D_SMA; symbol Device:D_Small -> Device:D_Schottky_Small; LCSC C64898 -> C2480
- J10: value Micro_SD_Card_Det2 -> Memory Card Slot
- U12: value SN74LVC1G18DBVR-TP -> SN74LVC1G3157DBVR; symbol shpc_ic:SN74LVC1G18 -> shpc_ic:SN74LVC1G3157; LCSC C49333182 -> C10426
Connections:
- net 3V3: now also R70.1, R71.1, R72.1
- net BTN_D: now also D7.1 (K); no longer R21.1
- net GND: now also C58.2, SW12.2, SW13.2
- net HSLCD_DC: now also U12.3 (B1); no longer U12.6 (Y0)
- net HSLCD_DCCK: now also U12.4 (A); no longer U12.3 (A)
- net HSLCD_SPIEN: now also U12.6 (S); no longer U12.1 (S)
- net HSSPI_MISO: no longer J4.14 (Pin_14), TP14.1
- net HSSPI_SCK: now also U12.1 (B2); no longer U12.4 (Y1)
- net LCA0: now also R73.1; no longer U7.49 (GPIO40/ADC0)
- net LCTF_ENX: now also TP26.1, U7.47 (GPIO38); no longer U4.17 (IO1_4)
- net VBAT: now also Q5.2 (S), C58.1; no longer Q5.3 (D)
- net VSYS: now also R9.2, C59.1; no longer R9.1
- net at J10.1 (DAT2): now also R71.2
- net HSTF_DETX: now reaches J10.10 (DET_A)
- net HSTF_DETX: now also TP24.1, U7.53 (GPIO42/ADC2), R70.2
- net at J10.8 (DAT1): now also R72.2
- net at J3.1 (Pin_1): now also U4.15 (IO1_2); no longer U4.13 (IO1_0)
- net at U4.14 (IO1_1): now also SW13.1; no longer J2.1 (Pin_1)
- net at SW6.1: now also U4.17 (IO1_4); no longer U4.15 (IO1_2)
- net at U4.16 (IO1_3): now also J2.1 (Pin_1)
- net at R12.1: now also Q5.3 (D); no longer Q5.2 (S)
- new net: C59.2, Q3.1 (G), R74.1
- new net: Q2.3 (D), R74.2, R9.1
- new net: R73.2, U7.49 (GPIO40/ADC0)
- new net: D7.2 (A), R21.1
- new net: SW12.1, U4.13 (IO1_0)
- new net HSLCD_MISO: J4.14 (Pin_14), TP14.1
- no-connect marks 18 -> 16
Other:
- note added: "inrush current protection"
- moved on the sheet: C1, D3, D6, J1, J2, J3, Q3, Q5, R21, R3, R4, R67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

Commit message: wip
Parts:
- removed SW1: GT-TC018A-H0375-L1, shpc_mechanical:GT-TC018A-H0375-L1, symbol shpc_mechanical:SKRPACE010
- added SW1: GT-TC018A-H0375-L1, shpc_mechanical:GT-TC018A-H0375-L1, symbol Switch:SW_Push_Shielded
- C49: value 10n -> 100n; LCSC C15849 -> C1691; URL https://www.lcsc.com/product-detail/C15849.html -> https://www.lcsc.com/product-detail/C1691.html
- J1: symbol Connector_Generic:Conn_01x02 -> Connector_Generic_MountingPin:Conn_01x02_MountingPin
- J11: footprint shpc_mechanical:PinSocket_2x12_P2.54mm_Horizontal -> Connector_PinSocket_2.54mm:PinSocket_2x12_P2.54mm_Horizontal
- J4: symbol Connector_Generic:Conn_01x40 -> Connector_Generic_MountingPin:Conn_01x40_MountingPin; now in the parts list
- J8: value AudioJack3_SwitchTR -> PJ-316A-6A; symbol Connector_Audio:AudioJack3_SwitchTR -> Connector_Audio:AudioJack4_SwitchTR1
- U13: footprint Package_SO:TSSOP-20-1EP_4.4x6.5mm_P0.65mm_EP2.15x3.35mm -> Package_SO:TSSOP-20_4.4x6.5mm_P0.65mm
Connections:
- net GND: now also C49.2, J1.MP (MountPin), J4.MP (MountPin), SW1.2, SW1.SH (B); no longer C49.1
- net at R5.2, U2.3 (SW): now also SW1.1
- net at Q6.1 (G), R61.2: now also C49.1, J8.R1N; no longer C49.2, J8.RN
- net at C48.2, R60.1: now also J8.R1; no longer J8.R
- no-connect marks 16 -> 17
Other:
- moved on the sheet: C3, R18, R19, R20, R5, R6, R7, TP10, TP11, TP12, TP13, TP14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
