File: kicad/host_shell.kicad_sch (KiCad schematic)
At the start: 232 parts, among them J1 FG PH-2AWT, J10 Memory Card Slot, J11 Conn_02x12_Odd_Even, J2 Conn_01x02, J3 Conn_01x02, J4 Conn_01x40, J5 Conn_02x10_Odd_Even, J6 Conn_01x03, J7 Conn_01x02, J8 PJ-316A-6A, J9 Conn_01x02, P1 TYPE-C16PIN, Q1 IRLML2246TRPBF, Q2 BSS138W, Q3 IRLML2246TRPBF, Q4 BSS138W, Q5 BSS84W, Q6 BSS138W, Q7 BSS138W, SW1 GT-TC018A-H0375-L1, SW10 Rubber, SW11 SKRPACE010_6, SW12 Rubber, SW13 Rubber, SW2 Rubber, SW3 Rubber, SW4 Rubber, SW5 Rubber, SW6 Rubber, SW7 Rubber, SW8 Rubber, SW9 Rubber, U1 MCP73831-2-OT, U10 LM4880MX/NOPB, U11 LM4890S, U12 SN74LVC1G3157DBVR, U13 SN74AHC541PWR, U2 XC6194AA03ER-G, U3 TPS63802, U4 PCA9555PW, U5 W25Q32JVSSIQ, U6 APS6404L-3SQRx-SN, U7 RP2350B, U8 74LVC2G17GW, U9 LM4890S, Y1 ABM8-272-T3

Commit message: wip
Parts:
- R15: value 511k -> 56k; LCSC C64042 -> C23206
- R16: value 91k -> 10k; LCSC C1161 -> C25744; URL https://www.lcsc.com/product-detail/C17168.html -> -- ミックスされた値 --
Changed lines of the file:
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@@
 	)
 	(symbol
+		(lib_id "Device:R_Small")
+		(at 185.42 91.44 0)
+		(unit 1)
+		(body_style 1)
+		(exclude_from_sim no)
+		(in_bom yes)
+		(on_board yes)
+		(in_pos_files yes)
+		(dnp no)
+		(property "Reference" "R16"
+			(at 186.69 90.678 0)
+			(show_name no)
+			(do_not_autoplace no)
+			(effects
+				(font
+					(size 1.27 1.27)
+				)
+				(justify left)
+			)
+		)
+		(property "Value" "10k"
+			(at 186.69 92.456 0)
+			(show_name no)
+			(do_not_autoplace no)
+			(effects
+				(font
+					(size 1.27 1.27)
+				)
+				(justify left)
+			)
+		)
+		(property "Footprint" "Resistor_SMD:R_0402_1005Metric"
+			(at 185.42 91.44 0)
+			(hide yes)
+			(show_name no)
+			(do_not_autoplace no)
+			(effects
+				(font
+					(size 1.27 1.27)
+				)
+			)
+		)
+		(property "Datasheet" ""
+			(at 185.42 91.44 0)
+			(hide yes)
+			(show_name no)
+			(do_not_autoplace no)
+			(effects
+				(font
+					(size 1.27 1.27)
+				)
+			)
+		)
+		(property "Description" "Resistor, small symbol"
+			(at 185.42 91.44 0)
+			(hide yes)
+			(show_name no)
+			(do_not_autoplace no)
+			(effects
+				(font
+					(size 1.27 1.27)
+				)
+			)
+		)
+		(property "LCSC" "C25744"
+			(at 187.96 90.1699 0)
+			(hide yes)
+			(show_name no)
+			(do_not_autoplace no)
+			(effects
+				(font
+					(size 1.27 1.27)
+				)
+			)
+		)
+		(property "URL" "-- ミックスされた値 --"
+			(at 187.96 90.1699 0)
+			(hide yes)
+			(show_name no)
+			(do_not_autoplace no)
+			(effects
+				(font
+					(size 1.27 1.27)
+				)
+			)
+		)
+		(pin "1"
+		)
+		(pin "2"
+		)
+		(instances
+			(project "host_shell"
+				(path "/5e0c6c36-a1dc-429a-ac71-852781b1edf9"
+					(reference "R16")
+					(unit 1)
+				)
+			)
+		)
+	)
+	(symbol
 		(lib_id "power:+3V3")
 		(at 246.38 205.74 0)
@@
 			)
 		)
-		(property "Value" "511k"
+		(property "Value" "56k"
 			(at 186.69 82.296 0)
 			(show_name no)
@@
 			)
 		)
-		(property "LCSC" "C64042"
+		(property "LCSC" "C23206"
 			(at 187.96 80.0099 0)
 			(hide yes)
@@
 					(unit 1)
 				)
-			)
-		)
-	)
-	(symbol
-		(lib_id "Device:R_Small")
-		(at 185.42 91.44 0)
-		(unit 1)
-		(body_style 1)
-		(exclude_from_sim no)
-		(in_bom yes)
-		(on_board yes)
-		(in_pos_files yes)
-		(dnp no)
-		(property "Reference" "R16"
-			(at 186.69 90.678 0)
-			(show_name no)
-			(do_not_autoplace no)
-			(effects
-				(font
-					(size 1.27 1.27)
-				)
-				(justify left)
-			)
-		)
-		(property "Value" "91k"
-			(at 186.69 92.456 0)
-			(show_name no)
-			(do_not_autoplace no)
-			(effects
-				(font
-					(size 1.27 1.27)
-				)
-				(justify left)
-			)
-		)
-		(property "Footprint" "Resistor_SMD:R_0402_1005Metric"
-			(at 185.42 91.44 0)
-			(hide yes)
-			(show_name no)
-			(do_not_autoplace no)
-			(effects
-				(font
-					(size 1.27 1.27)
-				)
-			)
-		)
-		(property "Datasheet" ""
-			(at 185.42 91.44 0)
-			(hide yes)
-			(show_name no)
-			(do_not_autoplace no)
-			(effects
-				(font
-					(size 1.27 1.27)
-				)
-			)
-		)
-		(property "Description" "Resistor, small symbol"
-			(at 185.42 91.44 0)
-			(hide yes)
-			(show_name no)
-			(do_not_autoplace no)
-			(effects
-				(font
-					(size 1.27 1.27)
-				)
-			)
-		)
-		(property "LCSC" "C1161"
-			(at 187.96 90.1699 0)
-			(hide yes)
-			(show_name no)
-			(do_not_autoplace no)
-			(effects
-				(font
-					(size 1.27 1.27)
-				)
-			)
-		)
-		(property "URL" "https://www.lcsc.com/product-detail/C17168.html"
-			(at 187.96 90.1699 0)
-			(hide yes)
-			(show_name no)
-			(do_not_autoplace no)
-			(effects
-				(font
-					(size 1.27 1.27)
-				)
-			)
-		)
-		(pin "1"
-		)
-		(pin "2"
-		)
-		(instances
-			(project "host_shell"
-				(path "/5e0c6c36-a1dc-429a-ac71-852781b1edf9"
-					(reference "R16")
-					(unit 1)
-				)

Commit message: add RTC
Parts:
- removed Q2: BSS138W, Package_TO_SOT_SMD:SOT-323_SC-70, symbol Transistor_FET:BSS138
- removed Q3: IRLML2246TRPBF, Package_TO_SOT_SMD:SOT-23, symbol Transistor_FET:Q_PMOS_GSD
- removed R9: 100k, Resistor_SMD:R_0402_1005Metric, symbol Device:R_Small
- added C60, C61: 100n, Capacitor_SMD:C_0402_1005Metric, symbol Device:C_Small
- added D8: SESD5Z5V, Diode_SMD:D_SOD-523, symbol Device:D_TVS_Small
- added D9: LBAT54HT1G, Diode_SMD:D_SOD-323, symbol Device:D_Schottky_Small
- added F1, F2: SMD1206P150TF, Fuse:Fuse_1206_3216Metric, symbol Device:Polyfuse_Small
- added R75: 10k, Resistor_SMD:R_0402_1005Metric, symbol Device:R_Small
- added R76: 100k, Resistor_SMD:R_0402_1005Metric, symbol Device:R_Small
- added TP41, TP42, TP43: TestPoint_Small, TestPoint:TestPoint_Pad_D1.0mm, symbol Connector:TestPoint_Small
- added U14: TPS22919DCKR, Package_TO_SOT_SMD:SOT-363_SC-70-6, symbol shpc_ic:TPS22919DCKR
- added U15: RV-3028-C7, Package_SON:MicroCrystal_C7_SON-8_1.5x3.2mm_P0.9mm, symbol Timer_RTC:RV-3028-C7
- C36, C37: footprint Capacitor_SMD:C_0603_1608Metric -> Capacitor_SMD:C_0402_1005Metric; LCSC C15849 -> C15195
- C38, C39, C43, C44, C45, C50, C51: footprint Capacitor_SMD:C_0603_1608Metric -> Capacitor_SMD:C_0402_1005Metric; LCSC C15849 -> C52923
- C41, C46, C49, C53: footprint Capacitor_SMD:C_0603_1608Metric -> Capacitor_SMD:C_0402_1005Metric; LCSC C1691 -> C1525
- C59: value 100n -> 1u; LCSC C1525 -> C52923; URL (none) -> https://www.lcsc.com/product-detail/C15849.html
- J4: footprint Connector_FFC-FPC:TE_4-1734839-0_1x40-1MP_P0.5mm_Horizontal -> shpc_mechanical:FFC_Conn_40P_Top_Hand; now left out of the parts list
- R4: value 22k -> 10k; LCSC C25768 -> C25744; URL https://www.lcsc.com/product-detail/C25768.html -> -- ミックスされた値 --
- R74: value 10k -> 100; LCSC C25744 -> C25076; URL -- ミックスされた値 -- -> (none)
Connections:
- net 3V3: now also C61.2, R76.2, U15.7 (VDD)
- net GND: now also C59.1, C60.1, C61.1, D8.2 (A2), R75.2, U14.2 (GND), U15.5 (VSS)
- net HSAUX_SCL: now also U15.3 (SCL)
- net HSAUX_SDA: now also U15.4 (SDA)
- net LCVSYS: now also R74.2, U14.6 (VOUT)
- net LCVSYSEN: now also U14.3 (ON)
- net VBAT: now also C60.2, F2.1, U15.6 (VBACKUP); no longer J1.1 (Pin_1)
- net VBUS: now also D8.1 (A1), F1.2; no longer P1.A4 (VBUS), P1.A9 (VBUS), P1.B4 (VBUS), P1.B9 (VBUS)
- net VSYS: now also C59.2, U14.1 (VIN); no longer C59.1
- net at R74.1: now also U14.5 (QOD); no longer C59.2
- net BTN_PWRX: now reaches R5.2, SW1.1, U2.3 (SW)
- net BTN_PWRX: now also TP23.1, D9.1 (K)
- net at U7.52 (GPIO41/ADC1): now also D9.2 (A), R76.1; no longer TP23.1
- new net: R75.1, TP41.1, U15.8 (EVI)
- new net: TP42.1, U15.1 (CLKOUT)
- new net: F1.1, P1.A4 (VBUS), P1.A9 (VBUS), P1.B4 (VBUS), P1.B9 (VBUS)
- new net: F2.2, J1.1 (Pin_1)
- new net: TP43.1, U15.2 (~{INT})
Other:
- note removed: "inrush current protection"
- moved on the sheet: C1, C56, C58, D1, D2, D3, D6, J5, P1, R1, R2, R3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
