File: kicad/host_shell.kicad_sch (KiCad schematic)
At the start: 238 parts, among them J1 FG PH-2AWT, J10 Memory Card Slot, J11 Conn_02x12_Odd_Even, J2 Conn_01x02, J3 Conn_01x02, J4 Conn_01x40, J5 Conn_02x10_Odd_Even, J6 Conn_01x03, J7 Conn_01x02, J8 PJ-316A-6A, J9 Conn_01x02, P1 TYPE-C16PIN, Q1 IRLML2246TRPBF, Q4 BSS138W, Q5 BSS84W, Q6 BSS138W, Q7 BSS138W, SW1 GT-TC018A-H0375-L1, SW10 PTS645SL50SMTR92, SW11 SKRPACE010_6, SW12 PTS645SL50SMTR92, SW13 PTS645SL50SMTR92, SW2 PTS645SL50SMTR92, SW3 PTS645SL50SMTR92, SW4 PTS645SL50SMTR92, SW5 PTS645SL50SMTR92, SW6 PTS645SL50SMTR92, SW7 PTS645SL50SMTR92, SW8 PTS645SL50SMTR92, SW9 PTS645SL50SMTR92, U1 MCP73831-2-OT, U10 LM4880MX/NOPB, U11 LM4890S, U12 SN74LVC1G3157DBVR, U13 SN74AHC541PWR, U14 TPS22919DCKR, U15 RV-3028-C7, U2 XC6194AA03ER-G, U3 TPS63802, U4 PCA9555PW, U5 W25Q32JVSSIQ, U6 APS6404L-3SQRx-SN, U7 RP2350B, U8 74LVC2G17GW, U9 LM4890S, Y1 ABM8-272-T3

Commit message: fix footprint
Parts:
- Q7: symbol Simulation_SPICE:NMOS -> Transistor_FET:BSS138
- R15: LCSC C23206 -> C25567
- RV1, U15: now not fitted; now left out of the parts list
- SW2: now in the parts list
Connections:
- net GND: now also Q7.2 (S); no longer Q7.3 (S)
- net HSLCD_BL_K: now also Q7.3 (D); no longer Q7.1 (D)
- net at R64.2, R65.1: now also Q7.1 (G); no longer Q7.2 (G)
Changed lines of the file:
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@@
 	)
 	(symbol
-		(lib_name "SKRPACE010_4")
+		(lib_name "SKRPACE010_1")
 		(lib_id "shpc_mechanical:SKRPACE010")
 		(at 344.17 38.1 0)
@@
 			)
 		)
-		(property "LCSC" "C23206"
+		(property "LCSC" "C25567"
 			(at 187.96 80.0099 0)
 			(hide yes)
@@
 	)
 	(symbol
-		(lib_name "SKRPACE010_3")
+		(lib_name "SKRPACE010_7")
 		(lib_id "shpc_mechanical:SKRPACE010")
 		(at 320.04 33.02 0)
@@
 		(body_style 1)
 		(exclude_from_sim no)
-		(in_bom no)
+		(in_bom yes)
 		(on_board yes)
 		(in_pos_files yes)
 		(dnp yes)
 		(property "Reference" "SW2"
-			(at 319.532 22.606 0)
+			(at 316.23 22.606 0)
 			(show_name no)
 			(do_not_autoplace no)
@@
 		)
 		(property "Value" "PTS645SL50SMTR92"
-			(at 320.294 22.606 0)
+			(at 316.992 22.606 0)
 			(show_name no)
 			(do_not_autoplace no)
@@
 		(dnp yes)
 		(property "Reference" "SW3"
-			(at 319.532 24.638 0)
+			(at 316.23 24.638 0)
 			(show_name no)
 			(do_not_autoplace no)
@@
 		)
 		(property "Value" "PTS645SL50SMTR92"
-			(at 320.294 24.638 0)
+			(at 316.992 24.638 0)
 			(show_name no)
 			(do_not_autoplace no)
@@
 			)
 		)
-		(property "Description" "-- ミックスされた値 --"
+		(property "Description" "50V Vds, 0.22A Id, N-Channel MOSFET, SOT-23"
 			(at 292.1 175.26 0)
 			(hide yes)
@@
 	)
 	(symbol
-		(lib_id "Simulation_SPICE:NMOS")
+		(lib_id "Transistor_FET:BSS138")
 		(at 383.54 185.42 0)
 		(unit 1)
@@
 		)
 		(property "Footprint" "Package_TO_SOT_SMD:SOT-323_SC-70"
-			(at 388.62 182.88 0)
+			(at 388.62 187.325 0)
 			(hide yes)
 			(show_name no)
@@
 				(font
 					(size 1.27 1.27)
+					(italic yes)
 				)
+				(justify left)
 			)
 		)
 		(property "Datasheet" "https://www.onsemi.com/pub/Collateral/BSS138-D.PDF"
-			(at 383.54 198.12 0)
+			(at 388.62 189.23 0)
 			(hide yes)
 			(show_name no)
@@
 					(size 1.27 1.27)
 				)
+				(justify left)
 			)
 		)
-		(property "Description" "-- ミックスされた値 --"
+		(property "Description" "50V Vds, 0.22A Id, N-Channel MOSFET, SOT-23"
 			(at 383.54 185.42 0)
 			(hide yes)
@@
 			)
 		)
-		(property "Description" "-- ミックスされた値 --"
+		(property "Description" "50V Vds, 0.22A Id, N-Channel MOSFET, SOT-23"
 			(at 81.28 88.9 0)
 			(hide yes)
@@
 	)
 	(symbol
-		(lib_name "SKRPACE010_5")
+		(lib_name "SKRPACE010_2")
 		(lib_id "shpc_mechanical:SKRPACE010")
 		(at 344.17 43.18 0)
@@
 	)
 	(symbol
-		(lib_name "SKRPACE010_1")
+		(lib_name "SKRPACE010_3")
 		(lib_id "shpc_mechanical:SKRPACE010")
 		(at 320.04 48.26 0)
@@
 		(dnp yes)
 		(property "Reference" "SW5"
-			(at 319.532 28.702 0)
+			(at 316.23 28.702 0)
 			(show_name no)
 			(do_not_autoplace no)
@@
 		)
 		(property "Value" "PTS645SL50SMTR92"
-			(at 320.294 28.702 0)
+			(at 316.992 28.702 0)
 			(show_name no)
 			(do_not_autoplace no)
@@
 		(body_style 1)
 		(exclude_from_sim no)
-		(in_bom yes)
+		(in_bom no)
 		(on_board yes)
 		(in_pos_files yes)
-		(dnp no)
+		(dnp yes)
 		(property "Reference" "RV1"
 			(at 288.798 116.078 90)
@@
 	)
 	(symbol
-		(lib_name "SKRPACE010_7")
+		(lib_name "SKRPACE010_4")
 		(lib_id "shpc_mechanical:SKRPACE010")
 		(at 344.17 33.02 0)
@@
 	)
 	(symbol
-		(lib_name "SKRPACE010_2")
+		(lib_name "SKRPACE010_5")
 		(lib_id "shpc_mechanical:SKRPACE010")
 		(at 320.04 43.18 0)
@@
 		(dnp yes)
 		(property "Reference" "SW4"
-			(at 319.532 26.67 0)
+			(at 316.23 26.67 0)
 			(show_name no)
 			(do_not_autoplace no)
@@
 		)
 		(property "Value" "PTS645SL50SMTR92"
-			(at 320.294 26.67 0)
+			(at 316.992 26.67 0)
 			(show_name no)
 			(do_not_autoplace no)
@@
 		(body_style 1)
 		(exclude_from_sim no)
-		(in_bom yes)
+		(in_bom no)
 		(on_board yes)
 		(in_pos_files yes)
-		(dnp no)
+		(dnp yes)
 		(property "Reference" "U15"
 			(at 49.022 271.018 0)
