File: kicad/host_shell.kicad_pcb (KiCad board)
At the start: 2 copper layers, 234 parts, among them J1 FG PH-2AWT, J10 Memory Card Slot, J11 Conn_02x12_Odd_Even, J2 Conn_01x02, J3 Conn_01x02, J4 Conn_01x40, J5 Conn_02x10_Odd_Even, J6 Conn_01x03, J7 Conn_01x02, J8 PJ-316A-6A, J9 Conn_01x02, P1 TYPE-C16PIN, Q1 IRLML2246TRPBF, Q2 BSS138W, Q3 IRLML2246TRPBF, Q4 BSS138W, Q5 BSS84W, Q6 BSS138W, Q7 BSS138W, SW1 GT-TC018A-H0375-L1, SW10 Rubber, SW11 SKRPACE010_6, SW12 Rubber, SW13 Rubber, SW2 Rubber, SW3 Rubber, SW4 Rubber, SW5 Rubber, SW6 Rubber, SW7 Rubber, SW8 Rubber, SW9 Rubber, U1 MCP73831-2-OT, U10 LM4880MX/NOPB, U11 LM4890S, U12 SN74LVC1G3157DBVR, U13 SN74AHC541PWR, U2 XC6194AA03ER-G, U3 TPS63802, U4 PCA9555PW, U5 W25Q32JVSSIQ, U6 APS6404L-3SQRx-SN, U7 RP2350B, U8 74LVC2G17GW, U9 LM4890S, Y1 ABM8-272-T3

Commit message: wip
Parts:
- R15: value 511k -> 56k
- R16: value 91k -> 10k
- moved C49 140.3 mm to (56.7, 129.7)
- moved R16 7.14 mm to (96.9, 88.5)
Changed lines of the file:
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@@
 		)
 	)
-	(footprint "Resistor_SMD:R_0402_1005Metric"
-		(layer "F.Cu")
-		(at 103.965 87.815)
-		(descr "Resistor SMD 0402 (1005 Metric), square (rectangular) end terminal, IPC-7351 nominal, (Body size source: IPC-SM-782 page 72, https://www.pcb-3d.com/wordpress/wp-content/uploads/ipc-sm-782a_amendment_1_and_2.pdf)")
-		(tags "resistor")
-		(property "Reference" "R16"
-			(at 0 -1.17 0)
-			(layer "F.SilkS")
-			(effects
-				(font
-					(size 1 1)
-					(thickness 0.15)
-				)
-			)
-		)
-		(property "Value" "91k"
-			(at 0 1.17 0)
-			(layer "F.Fab")
-			(effects
-				(font
-					(size 1 1)
-					(thickness 0.15)
-				)
-			)
-		)
-		(property "Datasheet" ""
-			(at 0 0 0)
-			(layer "F.Fab")
-			(hide yes)
-			(effects
-				(font
-					(size 1.27 1.27)
-				)
-			)
-		)
-		(property "Description" "Resistor, small symbol"
-			(at 0 0 0)
-			(layer "F.Fab")
-			(hide yes)
-			(effects
-				(font
-					(size 1.27 1.27)
-				)
-			)
-		)
-		(property "KiLib_Generator" "SMD_2terminal_chip_molded"
-			(at 0 0 0)
-			(layer "F.SilkS")
-			(hide yes)
-			(effects
-				(font
-					(size 1 1)
-					(thickness 0.15)
-				)
-			)
-		)
-		(property "LCSC" "C1161"
-			(at 0 0 0)
-			(unlocked yes)
-			(layer "F.Fab")
-			(hide yes)
-			(effects
-				(font
-					(size 1 1)
-					(thickness 0.15)
-				)
-			)
-		)
-		(property "URL" "https://www.lcsc.com/product-detail/C17168.html"
-			(at 0 0 0)
-			(unlocked yes)
-			(layer "F.Fab")
-			(hide yes)
-			(effects
-				(font
-					(size 1 1)
-					(thickness 0.15)
-				)
-			)
-		)
-		(property ki_fp_filters "R_*")
-		(sheetname "/")
-		(sheetfile "host_shell.kicad_sch")
-		(units
-			(unit
-				(name "A")
-				(pins "1" "2")
-			)
-		)
-		(attr smd)
-		(duplicate_pad_numbers_are_jumpers no)
-		(fp_line
-			(start -0.153641 -0.38)
-			(end 0.153641 -0.38)
-			(stroke
-				(width 0.12)
-				(type solid)
-			)
-			(layer "F.SilkS")
-		)
-		(fp_line
-			(start -0.153641 0.38)
-			(end 0.153641 0.38)
-			(stroke
-				(width 0.12)
-				(type solid)
-			)
-			(layer "F.SilkS")
-		)
-		(fp_rect
-			(start -0.93 -0.47)
-			(end 0.93 0.47)
-			(stroke
-				(width 0.05)
-				(type solid)
-			)
-			(fill no)
-			(layer "F.CrtYd")
-		)
-		(fp_rect
-			(start -0.525 -0.27)
-			(end 0.525 0.27)
-			(stroke
-				(width 0.1)
-				(type solid)
-			)
-			(fill no)
-			(layer "F.Fab")
-		)
-		(fp_text user "${REFERENCE}"
-			(at 0 0 0)
-			(layer "F.Fab")
-			(effects
-				(font
-					(size 0.26 0.26)
-					(thickness 0.04)
-				)
-			)
-		)
-		(pad "1" smd roundrect
-			(at -0.51 0)
-			(size 0.54 0.64)
-			(layers "F.Cu" "F.Mask" "F.Paste")
-			(roundrect_rratio 0.25)
-			(net "Net-(U3-FB)")
-			(pintype "passive")
-		)
-		(pad "2" smd roundrect
-			(at 0.51 0)
-			(size 0.54 0.64)
-			(layers "F.Cu" "F.Mask" "F.Paste")
-			(roundrect_rratio 0.25)
-			(net "GND")
-			(pintype "passive")
-		)
-		(embedded_fonts no)
-		(model "${KICAD10_3DMODEL_DIR}/Resistor_SMD.3dshapes/R_0402_1005Metric.step"
-			(offset
-				(xyz 0 0 0)
-			)
-			(scale
-				(xyz 1 1 1)
-			)
-			(rotate
-				(xyz 0 0 0)
-			)
-		)
-	)
 	(footprint "shpc_mechanical:SolderWirePad_1x02_SMD_150x50mil"
 		(layer "F.Cu")
@@
 			)
 		)
-		(property "Value" "511k"
+		(property "Value" "56k"
 			(at 0 1.17 0)
 			(layer "F.Fab")
@@
 			)
 		)
-		(property "LCSC" "C64042"
+		(property "LCSC" "C23206"
 			(at 0 0 0)
 			(unlocked yes)
@@
 		)
 	)
+	(footprint "Resistor_SMD:R_0402_1005Metric"
+		(layer "F.Cu")
+		(at 96.855 88.495)
+		(descr "Resistor SMD 0402 (1005 Metric), square (rectangular) end terminal, IPC-7351 nominal, (Body size source: IPC-SM-782 page 72, https://www.pcb-3d.com/wordpress/wp-content/uploads/ipc-sm-782a_amendment_1_and_2.pdf)")
+		(tags "resistor")
+		(property "Reference" "R16"
+			(at 0 -1.17 0)
+			(layer "F.SilkS")
+			(effects
+				(font
+					(size 1 1)
+					(thickness 0.15)
+				)
+			)
+		)
+		(property "Value" "10k"
+			(at 0 1.17 0)
+			(layer "F.Fab")
+			(effects
+				(font
+					(size 1 1)
+					(thickness 0.15)
+				)
+			)
+		)
+		(property "Datasheet" ""
+			(at 0 0 0)
+			(layer "F.Fab")
+			(hide yes)
+			(effects
+				(font
+					(size 1.27 1.27)
+				)
+			)
+		)
+		(property "Description" "Resistor, small symbol"
+			(at 0 0 0)
+			(layer "F.Fab")
+			(hide yes)
+			(effects
+				(font
+					(size 1.27 1.27)
+				)
+			)
+		)
+		(property "KiLib_Generator" "SMD_2terminal_chip_molded"
+			(at 0 0 0)
+			(layer "F.SilkS")
+			(hide yes)
+			(effects
+				(font
+					(size 1 1)
+					(thickness 0.15)
+				)
+			)
+		)
+		(property "LCSC" "C25744"
+			(at 0 0 0)
+			(unlocked yes)
+			(layer "F.Fab")
+			(hide yes)
+			(effects
+				(font
+					(size 1 1)
+					(thickness 0.15)
+				)
+			)
+		)
+		(property "URL" "-- ミックスされた値 --"
+			(at 0 0 0)
+			(unlocked yes)
+			(layer "F.Fab")
+			(hide yes)
+			(effects
+				(font
+					(size 1 1)
+					(thickness 0.15)
+				)
+			)
+		)
+		(property ki_fp_filters "R_*")
+		(sheetname "/")
+		(sheetfile "host_shell.kicad_sch")
+		(units
+			(unit
+				(name "A")
+				(pins "1" "2")
+			)
+		)
+		(attr smd)
+		(duplicate_pad_numbers_are_jumpers no)
+		(fp_line
+			(start -0.153641 -0.38)
+			(end 0.153641 -0.38)
+			(stroke
+				(width 0.12)
+				(type solid)
+			)
+			(layer "F.SilkS")
+		)
+		(fp_line
+			(start -0.153641 0.38)
+			(end 0.153641 0.38)
+			(stroke
+				(width 0.12)
+				(type solid)
+			)
+			(layer "F.SilkS")
+		)
+		(fp_rect
+			(start -0.93 -0.47)
+			(end 0.93 0.47)
+			(stroke
+				(width 0.05)
+				(type solid)
+			)
+			(fill no)
+			(layer "F.CrtYd")
+		)
+		(fp_rect
+			(start -0.525 -0.27)
+			(end 0.525 0.27)
+			(stroke
+				(width 0.1)
+				(type solid)
+			)
+			(fill no)
+			(layer "F.Fab")
+		)
+		(fp_text user "${REFERENCE}"
+			(at 0 0 0)
+			(layer "F.Fab")
+			(effects
+				(font
+					(size 0.26 0.26)
+					(thickness 0.04)
+				)
+			)
+		)
+		(pad "1" smd roundrect
+			(at -0.51 0)
+			(size 0.54 0.64)
+			(layers "F.Cu" "F.Mask" "F.Paste")
+			(roundrect_rratio 0.25)
+			(net "Net-(U3-FB)")
+			(pintype "passive")
+		)
+		(pad "2" smd roundrect
+			(at 0.51 0)
+			(size 0.54 0.64)
+			(layers "F.Cu" "F.Mask" "F.Paste")
+			(roundrect_rratio 0.25)
+			(net "GND")
+			(pintype "passive")
+		)
+		(embedded_fonts no)
+		(model "${KICAD10_3DMODEL_DIR}/Resistor_SMD.3dshapes/R_0402_1005Metric.step"
+			(offset
+				(xyz 0 0 0)
+			)
+			(scale
+				(xyz 1 1 1)
+			)
+			(rotate
+				(xyz 0 0 0)
+			)
+		)
+	)
 	(footprint "TestPoint:TestPoint_Pad_D1.0mm"
 		(layer "F.Cu")
@@
 	(footprint "Capacitor_SMD:C_0603_1608Metric"
 		(layer "F.Cu")
-		(at 1.505 0.755)
+		(at 56.725 129.7)
 		(descr "Capacitor SMD 0603 (1608 Metric), square (rectangular) end terminal, IPC-7351 nominal, (Body size source: IPC-SM-782 page 76, https://www.pcb-3d.com/wordpress/wp-content/uploads/ipc-sm-782a_amendment_1_and_2.pdf)")
 		(tags "capacitor")

Commit message: add RTC
Parts:
- added C59: 1u, Capacitor_SMD:C_0402_1005Metric, F.Cu at (256.5, 111.5)
- added C60: 100n, Capacitor_SMD:C_0402_1005Metric, F.Cu at (260.8, 109.7)
- added C61: 100n, Capacitor_SMD:C_0402_1005Metric, F.Cu at (256.5, 119.0)
- added D8: SESD5Z5V, Diode_SMD:D_SOD-523, F.Cu at (117.7, 136.0)
- added D9: LBAT54HT1G, Diode_SMD:D_SOD-323, F.Cu at (260.6, 121.7)
- added F1: SMD1206P150TF, Fuse:Fuse_1206_3216Metric, F.Cu at (120.0, 139.5)
- added F2: SMD1206P150TF, Fuse:Fuse_1206_3216Metric, F.Cu at (177.2, 111.0)
- added R4: 10k, Resistor_SMD:R_0402_1005Metric, F.Cu at (253.0, 113.7)
- added R74: 100, Resistor_SMD:R_0402_1005Metric, F.Cu at (253.0, 115.7)
- added R75: 10k, Resistor_SMD:R_0402_1005Metric, F.Cu at (253.0, 117.7)
- added R76: 100k, Resistor_SMD:R_0402_1005Metric, F.Cu at (253.0, 119.7)
- added TP41: TestPoint_Small, TestPoint:TestPoint_Pad_D1.0mm, F.Cu at (250.0, 114.2)
- added TP42: TestPoint_Small, TestPoint:TestPoint_Pad_D1.0mm, F.Cu at (250.0, 117.3)
- added TP43: TestPoint_Small, TestPoint:TestPoint_Pad_D1.0mm, F.Cu at (250.0, 120.3)
- added U14: TPS22919DCKR, Package_TO_SOT_SMD:SOT-363_SC-70-6, F.Cu at (256.4, 122.1)
- added U15: RV-3028-C7, Package_SON:MicroCrystal_C7_SON-8_1.5x3.2mm_P0.9mm, F.Cu at (260.6, 115.4)
- C36, C37, C38, C39, C41, C43, C44, C45, C46, C49, C50, C51, C53: footprint Capacitor_SMD:C_0603_1608Metric -> Capacitor_SMD:C_0402_1005Metric
- J4: footprint Connector_FFC-FPC:TE_4-1734839-0_1x40-1MP_P0.5mm_Horizontal -> shpc_mechanical:FFC_Conn_40P_Top_Hand; moved to B.Cu
- SW10, SW12, SW13, SW2, SW3, SW4, SW5, SW6, SW7, SW8, SW9: moved to B.Cu
- moved R56 212.6 mm to (-96.8, 71.8)
- moved C42 209.9 mm to (-82.0, 71.1)
- moved J7 208.8 mm to (-84.5, 64.5)
- moved C38 203.1 mm to (-91.9, 67.4)
- moved C39 203.1 mm to (-91.9, 69.9)
- moved C40 203.1 mm to (-91.9, 72.4)
- moved C41 198.6 mm to (-86.6, 71.6)
- moved U9 171.0 mm to (-92.2, 60.9)
- moved SW10 169.0 mm to (106.3, 214.8)
- moved SW2 169.0 mm to (83.2, 214.8)
- moved U11 156.8 mm to (227.4, 41.9)
- moved U10 156.7 mm to (30.4, 179.3), turned to 180 degrees
- moved Q2 152.1 mm to (205.5, 130.0)
- moved SW12 151.0 mm to (106.3, 205.6)
- moved SW3 151.0 mm to (83.2, 205.6)
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Connections:
- C58 pad 1: /VBAT -> VBAT
- J1 pad 1: /VBAT -> Net-(J1-Pin_1)
- P1 pad A4: VBUS -> Net-(F1-Pad1)
- P1 pad A9: VBUS -> Net-(F1-Pad1)
- P1 pad B4: VBUS -> Net-(F1-Pad1)
- P1 pad B9: VBUS -> Net-(F1-Pad1)
- Q1 pad 3: /VBAT -> VBAT
- Q5 pad 2: /VBAT -> VBAT
- R11 pad 1: /VBAT -> VBAT
- R5 pad 2: Net-(U2-SW) -> /BTN_PWRX
- SW1 pad 1: Net-(U2-SW) -> /BTN_PWRX
- TP23 pad 1: Net-(U7-GPIO41/ADC1) -> /BTN_PWRX
- U1 pad 3: /VBAT -> VBAT
- U2 pad 3: Net-(U2-SW) -> /BTN_PWRX
- U7 pad 52: Net-(U7-GPIO41/ADC1) -> Net-(D9-A)

Commit message: wip
Parts:
- removed C23: 100n, Capacitor_SMD:C_0402_1005Metric
- removed the C49 at (15.9, 156.5)
- removed the C59 at (220.0, 137.3)
- removed JP2, JP3, JP4: SolderJumper_3_Bridged12, Jumper:SolderJumper-3_P1.3mm_Bridged12_RoundedPad1.0x1.5mm
- removed Q2: BSS138W, Package_TO_SOT_SMD:SOT-323_SC-70
- removed Q3: IRLML2246TRPBF, Package_TO_SOT_SMD:SOT-23
- removed the R4 at (180.3, 119.5)
- removed the R74 at (198.5, 131.4)
- removed R9: 100k, Resistor_SMD:R_0402_1005Metric
- removed the SW1 at (233.3, 80.2)
- J2, J3: footprint shpc_mechanical:SolderWirePad_1x02_SMD_150x50mil -> shpc_mechanical:SolderWirePad_1x02_SMD_2.5x1.5mm
- J7, J9: footprint shpc_mechanical:SolderWirePad_1x02_SMD_150x50mil -> shpc_mechanical:SolderWirePad_2x01_SMD_2.5x1.5mm
- SW10, SW12, SW13, SW2, SW3, SW4, SW5, SW6, SW7, SW8, SW9: footprint shpc_mechanical:Rubber_Contact -> Button_Switch_SMD:SW_SPST_PTS645Sx43SMTR92
- TP21: moved to B.Cu
- moved D9 205.7 mm to (58.2, 84.6)
- moved C60 201.5 mm to (61.1, 136.7)
- moved U15 199.4 mm to (62.1, 134.8), turned to -90 degrees
- moved R76 195.3 mm to (61.0, 83.7), turned to -90 degrees
- moved C61 194.1 mm to (63.2, 136.7), turned to 180 degrees
- moved R75 189.2 mm to (64.6, 134.9), turned to 90 degrees
- moved TP43 187.8 mm to (62.6, 132.3), turned to -90 degrees
- moved TP42 185.9 mm to (64.7, 132.3), turned to -90 degrees
- moved TP41 185.0 mm to (66.2, 135.4), turned to -90 degrees
- moved R56 181.9 mm to (77.9, 122.6)
- moved C40 180.8 mm to (81.7, 122.7), turned to -90 degrees
- moved U9 179.9 mm to (77.7, 120.2)
- moved C39 175.7 mm to (75.6, 123.0), turned to -90 degrees
- moved C41 175.0 mm to (81.5, 120.2), turned to 90 degrees
- moved C38 173.5 mm to (73.5, 119.9), turned to 180 degrees
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Connections:
- J10 pad 10: /HSTF_DETX -> GND
- J10 pad 9: GND -> /HSTF_DETX
- R45 pad 1: Net-(U7-GPIO25) -> Net-(U7-GPIO21)
- R46 pad 1: Net-(U7-GPIO26) -> Net-(U7-GPIO22)
- R50 pad 1: Net-(U8-1Y) -> Net-(U8-2Y)
- R51 pad 1: Net-(U8-2Y) -> Net-(U8-1Y)
- TP17 pad 1: /LCA0 -> Net-(U4-~{INT})
- U4 pad 1: unconnected-(U4-~{INT}-Pad1) -> Net-(U4-~{INT})
- U4 pad 2: Net-(JP3-C) -> GND
- U4 pad 21: Net-(JP2-C) -> 3V3
- U4 pad 3: Net-(JP4-C) -> GND
- U7 pad 21: /HSLCD_RSTX -> Net-(U7-GPIO21)
- U7 pad 22: /HSLCD_RDX -> Net-(U7-GPIO22)
- U7 pad 23: /HSLCD_WRX -> /HSLCD_RSTX
- U7 pad 25: /HSLCD_CSX -> /HSLCD_RDX
- U7 pad 26: Net-(U7-GPIO25) -> /HSLCD_WRX
- U7 pad 27: Net-(U7-GPIO26) -> /HSLCD_CSX
- U8 pad 1: /HSAUDIO_L -> /HSAUDIO_R
- U8 pad 3: /HSAUDIO_R -> /HSAUDIO_L
Routing:
- net 3V3: track 0.00 -> 531.5 mm, vias 0 -> 24
- net /BTN_PWRX: track 0.00 -> 128.0 mm, vias 0 -> 2
- net /HSSPI_SCK: track 0.00 -> 126.2 mm, vias 0 -> 4
- net /SPKEN: track 0.00 -> 121.1 mm, vias 0 -> 6
- net /HSTF_DETX: track 0.00 -> 120.4 mm
- net /HSSPI_MOSI: track 0.00 -> 120.2 mm, vias 0 -> 3
- net Net-(C44-Pad2): track 0.00 -> 117.4 mm, vias 0 -> 3
- net /BTN_D: track 0.00 -> 113.1 mm, vias 0 -> 2
- net /HSTF_CSX: track 0.00 -> 112.7 mm, vias 0 -> 5
- net /HSSPI_MISO: track 0.00 -> 105.7 mm
- net /EXTVIDENX: track 0.00 -> 101.9 mm, vias 0 -> 1
- net Net-(U4-IO0_2): track 0.00 -> 95.8 mm, vias 0 -> 1
- net A3V3: track 0.00 -> 93.8 mm, vias 0 -> 4
- net /SYSSD: track 0.00 -> 93.2 mm, vias 0 -> 2
- net /ADCBAT: track 0.00 -> 92.6 mm, vias 0 -> 2
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- added copper zone on B.Cu, net GND
- added copper zone on F.Cu, net GND
Other:
- board outline added: 90 x 100 mm

Commit message: wip
Parts:
- SW10, SW12, SW13, SW2, SW3, SW4, SW5, SW6, SW7, SW8, SW9: value Rubber -> PTS645SL50SMTR92
- moved TP22 16.5 mm to (58.3, 63.1)
- moved SW1 2.75 mm to (65.0, 54.8)
- moved D1 0.70 mm to (101.4, 141.2)
- moved D2 0.70 mm to (98.6, 141.2)
- moved R1 0.70 mm to (97.3, 143.0)
- moved R2 0.70 mm to (102.7, 143.0)
- moved TP1 0.70 mm to (101.1, 143.3)
- moved TP2 0.70 mm to (98.9, 143.3)
- moved TP4 0.63 mm to (107.6, 127.5)
- moved SW11 0.28 mm to (58.2, 68.3)
- moved C2 0.22 mm to (109.7, 133.1)
- moved R6 0.20 mm to (106.8, 130.6)
- moved U2 0.15 mm to (105.9, 132.8)
- moved R5 0.13 mm to (107.7, 133.1)
- moved C59 0.08 mm to (104.1, 134.1)
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Routing:
- net VBAT: track 31.1 -> 107.3 mm, vias 0 -> 4
- net Net-(U7-RUN): track 25.3 -> 28.8 mm
- net /BTN_PWRX: track 128.0 -> 125.6 mm
- net GND: track 38.9 -> 40.5 mm, vias 542 -> 593
- net Net-(U4-IO0_2): track 95.8 -> 95.0 mm
- net 3V3: track 531.5 -> 530.7 mm
- net Net-(P1-CC1): track 2.68 -> 3.40 mm
- net Net-(P1-CC2): track 2.44 -> 3.14 mm
Other:
- outline, holes or cut-outs redrawn

Commit message: layout review feeedback
Routing:
- net Net-(U4-IO1_1): track 25.0 -> 35.7 mm, vias 1 -> 3
- net Net-(U4-IO0_4): track 7.98 -> 18.6 mm, vias 1 -> 3
- net Net-(U4-IO0_7): track 14.4 -> 24.3 mm, vias 1 -> 3
- net Net-(U4-IO0_5): track 3.45 -> 13.2 mm
- net Net-(U4-IO1_4): track 21.8 -> 30.1 mm, vias 1 -> 3
- net Net-(U4-IO0_6): track 16.1 -> 24.1 mm
- net Net-(U4-IO0_2): track 95.0 -> 102.9 mm, vias 1 -> 3
- net Net-(U4-IO0_1): track 82.2 -> 90.2 mm
- net Net-(U4-IO0_0): track 82.1 -> 90.0 mm, vias 1 -> 3
- net Net-(U4-IO1_0): track 44.7 -> 52.1 mm, vias 1 -> 3
- net /BTN_D: track 113.1 -> 118.3 mm, vias 2 -> 3
- net /SPKEN: track 121.4 -> 123.5 mm
- net 3V3: track 530.7 -> 531.7 mm
- net GND: vias 593 -> 605

Commit message: add silks
Parts:
- added G***: LOGO, LOGO, F.Cu at (100.0, 90.0)
- added G***: LOGO, LOGO, F.Cu at (100.0, 72.0)
- TP10, TP11, TP12, TP13, TP14, TP28, TP29, TP30, TP31, TP32, TP9: moved to B.Cu
- moved TP9 9.77 mm to (91.3, 84.0)
- moved TP13 5.22 mm to (96.0, 71.4)
- moved TP11 4.64 mm to (96.0, 69.2)
- moved TP10 2.91 mm to (97.9, 68.1)
- moved TP12 2.14 mm to (97.9, 70.3)
Routing:
- net Net-(J4-Pin_1): track 3.65 -> 5.93 mm, vias 1 -> 0
- net Net-(J4-Pin_4): track 9.01 -> 7.21 mm, vias 1 -> 0
- net Net-(J4-Pin_2): track 6.51 -> 7.58 mm, vias 1 -> 0
- net Net-(R54-Pad2): track 19.7 -> 20.3 mm
- net /HSLCD_SPIEN: track 79.2 -> 79.4 mm, vias 3 -> 2
- net Net-(J4-Pin_3): track 5.56 -> 5.43 mm, vias 1 -> 0
- net GND: vias 605 -> 606
- net /HSLCD_MISO: vias 1 -> 0
Other:
- board text added: "3V3"
- board text added: "AUDIO_L"
- board text added: "AUDIO_R"
- board text added: "AUX_SCL"
- board text added: "AUX_SDA"
- board text added: "CSX"
- board text added: "D0"
- board text added: "D1"
- board text added: "D2"
- board text added: "D3"
- board text added: "D4"
- board text added: "D5"
- board text added: "D6"
- board text added: "D7"
- board text added: "DC"
- board text added: "ENX"
- board text added: "GND"
- board text added: "LCA0"
- board text added: "LCIO0"
- board text added: "LCIO1"
- board text added: "LCIO10"
- board text added: "LCIO11"
- board text added: "LCIO12"
- board text added: "LCIO13"
- board text added: "LCIO2"
- board text added: "LCIO3"
- board text added: "LCIO4"
- board text added: "LCIO5"
- board text added: "LCIO6"
- board text added: "LCIO7"
- board text added: "LCIO8"
- board text added: "LCIO9"
- board text added: "LCVSYS"
- board text added: "RDX"
- board text added: "RSTX"
- board text added: "USB_DM"
- board text added: "USB_DP"
- board text added: "VSYS"
- board text added: "WRX"
